Commit message: syncing urdfs across laptop and robot

File: src/robot_description/urdf/hexapod.urdf (robot description, URDF)
Before this commit: robot hexapod, 25 links, 24 joints
Links:
- link base_link: mass 0.786295693203365 -> 0.786295694888978
- link front_left_coxa_link: mass 0.086385 -> 0.086281
- link front_left_femur_link: mass 0.031609 -> 0.0314
- link front_left_foot_link: mass 0.0010269 -> 0.00102687106652255
- link front_right_coxa_link: mass 0.086385 -> 0.086281
- link front_right_femur_link: mass 0.03096 -> 0.030751
- link front_right_foot_link: mass 0.0010269 -> 0.00102687106652255
- link middle_left_coxa_link: mass 0.086385 -> 0.086281
- link middle_left_femur_link: mass 0.031609 -> 0.0314
- link middle_left_foot_link: mass 0.0010269 -> 0.00102687106652256
- link middle_right_coxa_link: mass 0.086385 -> 0.086281
- link middle_right_femur_link: mass 0.03096 -> 0.030751
- link middle_right_foot_link: mass 0.0010269 -> 0.00102687106652256
- link rear_left_coxa_link: mass 0.086385 -> 0.086281
- link rear_left_femur_link: mass 0.03096 -> 0.030751
- link rear_left_foot_link: mass 0.0010269 -> 0.00102687106652255
- link rear_right_coxa_link: mass 0.086385 -> 0.086281
- link rear_right_femur_link: mass 0.03096 -> 0.030751
- link rear_right_foot_link: mass 0.00102687106652255 -> 0.0010269
Joints:
- joint front_left_coxa_joint: axis -0.0001863 -7.2511E-05 -1 -> 0.0425207281634428 0.00387756005096805 -0.999088060285229; limit lower=-2.57 upper=2.57 effort=0 velocity=0 -> lower=-1.57 upper=1.57 effort=0 velocity=0; origin xyz=0.06114 0.061135 0.047119 rpy=0 0 0 -> xyz=0.0597794623037307 0.0610074569827942 0.0154258000000004 rpy=0 0 0
- joint front_left_femur_joint: limit lower=-2.57 upper=2.57 effort=0 velocity=0 -> lower=-1.57 upper=1.57 effort=0 velocity=0; origin xyz=0.071347 0.027719 -0.021317 rpy=-0.00010412 0.00010671 0.79764 -> xyz=0.0506354195835637 0.0493770568562628 0.0103729999999975 rpy=-0.000104123938980253 0.000104107183134694 0.785317693150283
- joint front_left_foot_joint: origin xyz=0.048031 0.031527 -0.1543 rpy=-0.063104 0.061486 -0.80158 -> xyz=-0.157028654923345 -0.000166190898608631 0.0381859537813213 rpy=-2.271181641943 -0.422454157208771 -1.23828061902425
- joint front_left_tibia_joint: limit lower=-2.57 upper=2.57 effort=0 velocity=0 -> lower=0 upper=3.1415 effort=0 velocity=0; origin xyz=0.083521 0 0.06927 rpy=-9.4214E-05 9.656E-05 5.5354E-05 -> xyz=0.108492266657861 0 -0.00133055426669743 rpy=0.000184555914276492 -0.000184623471871961 0.00026345026142038
- joint front_right_coxa_joint: axis 7.2511E-05 -0.0001863 1 -> -0.0437385357924751 0.00789225955945658 0.999011838130949; limit lower=-2.57 upper=2.57 effort=0 velocity=0 -> lower=-1.57 upper=1.57 effort=0 velocity=0; origin xyz=0.06114 -0.061135 0.047119 rpy=0 0 0 -> xyz=0.0597479377257695 -0.0608728713812492 0.0154258000000012 rpy=0 0 0
- joint front_right_femur_joint: limit lower=-2.57 upper=2.57 effort=0 velocity=0 -> lower=-1.57 upper=1.57 effort=0 velocity=0; origin xyz=0.034257 -0.068448 -0.021317 rpy=-0.00010412 -8.4145E-05 -0.67968 -> xyz=0.0506416297387538 -0.0495369568805863 0.0103729999999976 rpy=-0.000104123938883876 -0.000104140694039058 -0.785478611961186
- joint front_right_foot_joint: axis 0 -0.999997292508137 -0.00232700053339396 -> 0 0 0; origin xyz=0.0619475711858466 0.0315268097379976 -0.149260389779713 rpy=-0.00207607080041258 -0.00287997686253638 0.679644410877493 -> xyz=-0.157034797728908 -0.000166190898609997 0.0381606844208381 rpy=2.27095727607043 -0.422354608328963 1.23800658745024
- joint front_right_tibia_joint: limit lower=-2.57 upper=2.57 effort=0 velocity=0 -> lower=0 upper=3.1415 effort=0 velocity=0; origin xyz=0.015841 0 0.10735 rpy=-9.1062E-05 -7.3584E-05 3.7276E-05 -> xyz=0.10849 0 -0.0013531 rpy=0.00018461 0.00018454 0.00026348
- joint middle_left_coxa_joint: axis 0 0 -1 -> -8.04594058439077E-05 -0.000183005707343813 -0.999999980017597; limit lower=-2.57 upper=2.57 effort=0 velocity=0 -> lower=-1.57 upper=1.57 effort=0 velocity=0; origin xyz=0 0.086462 0.047119 rpy=-0.00018301 8.0459E-05 0 -> xyz=0 0.0864545384187688 0.0154258000000007 rpy=0 0 0
- joint middle_left_femur_joint: limit lower=-2.57 upper=2.57 effort=0 velocity=0 -> lower=-1.57 upper=1.57 effort=0 velocity=0; origin xyz=0.035286 0.067928 -0.021301 rpy=-0.00017502 0.001814 1.5188 -> xyz=2.10046607146265E-05 0.0696742115812287 0.0138198356843305 rpy=1.56394087721752 -1.46256545726282 0.00681533790492595
- joint middle_left_foot_joint: origin xyz=-0.015167 0.031527 -0.16089 rpy=-0.48384 0.00019266 -1.5708 -> xyz=0.15911554000758 -0.000166190898614748 0.0282561579362873 rpy=1.35669573662495 0 -1.57059641480066
- joint middle_left_tibia_joint: limit lower=-2.57 upper=2.57 effort=0 velocity=0 -> lower=0 upper=3.1415 effort=0 velocity=0; origin xyz=0.06729 0 0.085125 rpy=-8.855E-05 0.0017051 0.00013407 -> xyz=-0.00465888477440595 -0.000506201381017687 -0.108495899458512 rpy=0.000455617198050646 -1.15731885852398 0.107730800271824
- joint middle_right_coxa_joint: axis -8.0459E-05 -0.00018301 1 -> -8.04591239439089E-05 -0.000183005730591605 0.999999980017616; limit lower=-2.57 upper=2.57 effort=0 velocity=0 -> lower=-1.57 upper=1.57 effort=0 velocity=0; origin xyz=0 -0.086462 0.047119 rpy=0 0 0 -> xyz=0 -0.0864558000013206 0.0154258000001641 rpy=0 0 0
- joint middle_right_femur_joint: axis 0.044752 0.999 -0.00010412 -> 0 1 0; limit lower=-2.57 upper=2.57 effort=0 velocity=0 -> lower=-1.57 upper=1.57 effort=0 velocity=0; origin xyz=-0.034791 -0.068178 -0.021317 rpy=0 0 -1.5708 -> xyz=-2.04500179069247E-05 -0.0696729499986796 0.0103729999998343 rpy=-0.00017029088670727 0.912907710407541 -1.57101153482602
- joint middle_right_foot_joint: origin xyz=0.071308 0.028338 -0.14568 rpy=-0.057868 0.0025818 1.5706 -> xyz=0.159115539999232 -0.0001661908986167 0.0282561579833033 rpy=-1.35669573692048 0 1.57099623878914
- joint middle_right_tibia_joint: axis -0.044725 -0.999 0.00019256 -> 0 -1 0; limit lower=-2.57 upper=2.57 effort=0 velocity=0 -> lower=0 upper=3.1415 effort=0 velocity=0; origin xyz=0.040131 -0.0017945 0.1008 rpy=0 0 0 -> xyz=0.067399025687048 0 0.0850277227476781 rpy=-3.14148378102785 0.498689769885715 -3.14123342941393
- joint rear_left_coxa_joint: axis 0 0 -1 -> 0 0 0; limit lower=-2.57 upper=2.57 effort=0 velocity=0 -> lower=-1.57 upper=1.57 effort=0 velocity=0; origin xyz=-0.061135 0.06114 0.047119 rpy=-0.0001863 -7.2511E-05 0 -> xyz=-0.0625828215626599 0.0588152120207696 0.0154258000000006 rpy=0 0 0; type revolute -> fixed
- joint rear_left_femur_joint: limit lower=-2.57 upper=2.57 effort=0 velocity=0 -> lower=-1.57 upper=1.57 effort=0 velocity=0; origin xyz=-0.0069169 0.076233 -0.021302 rpy=-0.00013328 -0.00038067 2.0884 -> xyz=-0.0478016922764079 0.0515996698665222 0.0103730000000015 rpy=-0.00010412393892102 -0.000104140694076206 2.35611404162862
- joint rear_left_foot_joint: origin xyz=0.056346 0.031527 -0.15146 rpy=-0.033706 0.00019667 -1.5708 -> xyz=-0.157034797728908 -0.000166190898612381 0.0381606844208325 rpy=-2.1990344128274 -8.04446851697625E-05 -1.57097933897523
- joint rear_left_tibia_joint: limit lower=-2.57 upper=2.57 effort=0 velocity=0 -> lower=0 upper=3.1415 effort=0 velocity=0; origin xyz=0.040782 0 0.10055 rpy=-9.2524E-05 -0.0001625 4.4556E-05 -> xyz=0.108491987220254 0 -0.0013531475220351 rpy=0.000184610780237547 0.000184543218609282 0.000263479964488295
- joint rear_right_coxa_joint: axis 0 0 1 -> -0.00419160564654864 -0.0399618653751459 -0.999192413781171; limit lower=-2.57 upper=2.57 effort=0 velocity=0 -> lower=-1.57 upper=1.57 effort=0 velocity=0; origin xyz=-0.061135 -0.06114 0.047119 rpy=7.2511E-05 -0.0001863 0 -> xyz=-0.0609902962483643 -0.0598679792477214 0.0154257999999996 rpy=0 0 0
- joint rear_right_femur_joint: limit lower=-2.57 upper=2.57 effort=0 velocity=0 -> lower=-1.57 upper=1.57 effort=0 velocity=0; origin xyz=-0.075358 -0.013438 -0.021302 rpy=-0.00015016 -0.00012276 -2.5381 -> xyz=-0.049419532013472 -0.0505215882168034 0.0103730000000031 rpy=-0.000104123938777913 0.000104107182932361 -2.35627496043963
- joint rear_right_foot_joint: origin xyz=0.1098 0.031527 -0.11857 rpy=-0.2178 0.28534 2.4759 -> xyz=-0.157028654923349 -0.000166190898619894 0.0381859537813168 rpy=2.27118164194299 0.422454157208764 1.9033120345656
- joint rear_right_tibia_joint: axis 0 1 0 -> 0 -1 0; limit lower=-2.57 upper=2.57 effort=0 velocity=0 -> lower=0 upper=3.1415 effort=0 velocity=0; origin xyz=-0.016411 -1.2488E-05 0.10726 rpy=-6.4057E-05 4.4155E-05 -2.7619E-05 -> xyz=0.10849 0 -0.0013306 rpy=0.00018456 -0.00018462 0.00026345

Commit message: Inverse Kinematics are working with all of the legs and can be displayed in the URDF. The trajectory controller can send a multiarray of data and the legs can go to different points in space. Joint space seems good. Need to work on motor space, gaits, and standing next.

File: src/robot_description/urdf/hexapod.urdf (robot description, URDF)
Before this commit: robot Hexapod, 25 links, 24 joints
Joints:
- joint rear_left_coxa_joint: axis 0 0 0 -> 0 0 1; type fixed -> revolute
